File: hardware/geophone.kicad_sch (KiCad schematic)
At the start: 60 parts, among them J10 Screw_Terminal_01x06, J11 Conn_01x02_Socket, J12 Conn_01x02_Socket, J8 Screw_Terminal_01x04, J9 Conn_01x02_Socket, U10 OPA2211, U11 OPA2211, U12 OPA2211, U13 LM35-LP, U14 ADS1115IDGS, U15 ADS131M04, X1 8MHz

Commit message: Fix footprints
Parts:
- C68, C70, C71, C74: footprint Capacitor_SMD:CP_Elec_4x5.4 -> Capacitor_SMD:CP_Elec_4x5.7
Changed lines of the file:
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@@
       (effects (font (size 1.27 1.27)))
     )
-    (property "Footprint" "Capacitor_SMD:CP_Elec_4x5.4" (at 29.21 140.97 0)
+    (property "Footprint" "Capacitor_SMD:CP_Elec_4x5.7" (at 29.21 140.97 0)
       (effects (font (size 1.27 1.27)) hide)
     )
@@
       (effects (font (size 1.27 1.27)) (justify left))
     )
-    (property "Footprint" "Capacitor_SMD:CP_Elec_4x5.4" (at 29.845 98.425 0)
+    (property "Footprint" "Capacitor_SMD:CP_Elec_4x5.7" (at 29.845 98.425 0)
       (effects (font (size 1.27 1.27)) hide)
     )
@@
     (pin "1")
     (pin "8")
+    (pin "9")
     (instances
       (project "Explorer"
@@
     (pin "1")
     (pin "8")
+    (pin "9")
     (instances
       (project "Explorer"
@@
       (effects (font (size 1.27 1.27)))
     )
-    (property "Footprint" "Capacitor_SMD:CP_Elec_4x5.4" (at 85.09 140.97 0)
+    (property "Footprint" "Capacitor_SMD:CP_Elec_4x5.7" (at 85.09 140.97 0)
       (effects (font (size 1.27 1.27)) hide)
     )
@@
     (pin "1")
     (pin "8")
+    (pin "9")
     (instances
       (project "Explorer"
@@
     (pin "1")
     (pin "8")
+    (pin "9")
     (instances
       (project "Explorer"
@@
       (effects (font (size 1.27 1.27)) (justify left))
     )
-    (property "Footprint" "Capacitor_SMD:CP_Elec_4x5.4" (at 150.495 151.13 0)
+    (property "Footprint" "Capacitor_SMD:CP_Elec_4x5.7" (at 150.495 151.13 0)
       (effects (font (size 1.27 1.27)) hide)
     )
@@
     (pin "1")
     (pin "8")
+    (pin "9")
     (instances
       (project "Explorer"
@@
     (pin "1")
     (pin "8")
-    (instances
-      (project "Explorer"
+    (pin "9")
+    (instances
+      (project "Explorer"
